File: Hardware/pico_coaster.kicad_pcb (KiCad board)
At the start: 2 copper layers, 90 x 90 mm, 144 parts, among them J1 Conn_01x02, J2 Conn_01x02, J3 Conn_02x06_Odd_Even, J4 Conn_01x04, J5 USB_C_Receptacle_USB2.0, J6 Conn_01x02, SW2 SW_Push, SW3 SW_Push, SW4 SW_Push, SW5 SW_Push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

Commit message: update cap values in pcb file
Parts:
- C13, C14: value 20p -> 10p
